File: Hardware/MainPCB/Audio.kicad_sch (KiCad schematic)
At the start: 9 parts, among them U8 MAX4908

Commit message: Fixed color bending issue; Added diagnostics
Parts:
- R42, R43: footprint Resistor_SMD:R_0603_1608Metric -> RT5XP-EXP:R_0603; symbol Device:R -> RT5XP_EXP:R
- U8: footprint Package_DFN_QFN:TDFN-14-1EP_3x3mm_P0.4mm_EP1.78x2.35mm -> RT5XP-EXP:TDFN-14-1EP_3x3mm_P0.4mm_EP1.78x2.35mm; symbol AE:MAX4908 -> RT5XP_EXP:MAX4908
Changed lines of the file:
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@@
   (title_block
     (title "RT5XP-EXP")
-    (date "2023-04-07")
-    (rev "V1.1")
+    (date "2023-09-01")
+    (rev "V1.2")
     (company "Artjom Eske")
   )
@@
     (pin "2")
   )
-  (symbol (lib_id "Device:R") (at 185.42 104.14 180) (unit 1)
+  (symbol (lib_id "RT5XP_EXP:R") (at 185.42 104.14 180) (unit 1)
     (in_bom yes) (on_board yes)
     (property "Reference" "R43" (id 0) (at 189.23 102.87 0))
     (property "Value" "100R" (id 1) (at 189.23 105.41 0))
-    (property "Footprint" "Resistor_SMD:R_0603_1608Metric" (id 2) (at 187.198 104.14 90)
-      (effects (font (size 1.27 1.27)) hide)
-    )
-    (property "Datasheet" "~" (id 3) (at 185.42 104.14 0)
+    (property "Footprint" "RT5XP-EXP:R_0603" (id 2) (at 185.801 104.14 0)
+      (effects (font (size 1.27 1.27)) hide)
+    )
+    (property "Datasheet" "~" (id 3) (at 185.801 104.14 0)
       (effects (font (size 1.27 1.27)) hide)
     )
@@
     (pin "2")
   )
-  (symbol (lib_id "AE:MAX4908") (at 154.94 91.44 0) (unit 1)
+  (symbol (lib_id "RT5XP_EXP:MAX4908") (at 154.94 91.44 0) (unit 1)
     (in_bom yes) (on_board yes)
     (property "Reference" "U8" (id 0) (at 162.56 76.2 0)
@@
       (effects (font (size 1.27 1.27)) (justify left))
     )
-    (property "Footprint" "Package_DFN_QFN:TDFN-14-1EP_3x3mm_P0.4mm_EP1.78x2.35mm" (id 2) (at 165.1 78.74 0)
-      (effects (font (size 1.27 1.27)) hide)
-    )
-    (property "Datasheet" "" (id 3) (at 165.1 78.74 0)
+    (property "Footprint" "RT5XP-EXP:TDFN-14-1EP_3x3mm_P0.4mm_EP1.78x2.35mm" (id 2) (at 154.94 91.44 0)
+      (effects (font (size 1.27 1.27)) hide)
+    )
+    (property "Datasheet" "" (id 3) (at 154.94 91.44 0)
       (effects (font (size 1.27 1.27)) hide)
     )
@@
     (pin "9")
   )
-  (symbol (lib_id "Device:R") (at 176.53 104.14 180) (unit 1)
+  (symbol (lib_id "RT5XP_EXP:R") (at 176.53 104.14 180) (unit 1)
     (in_bom yes) (on_board yes)
     (property "Reference" "R42" (id 0) (at 180.34 102.87 0))
     (property "Value" "100R" (id 1) (at 180.34 105.41 0))
-    (property "Footprint" "Resistor_SMD:R_0603_1608Metric" (id 2) (at 178.308 104.14 90)
-      (effects (font (size 1.27 1.27)) hide)
-    )
-    (property "Datasheet" "~" (id 3) (at 176.53 104.14 0)
-      (effects (font (size 1.27 1.27)) hide)
-    )
+    (property "Footprint" "RT5XP-EXP:R_0603" (id 2) (at 176.911 104.14 0)
+      (effects (font (size 1.27 1.27)) hide)
+    )
+    (property "Datasheet" "~" (id 3) (at 176.911 104.14 0)
+      (effects (font (size 1.27 1.27)) hide)
+    )
